File: psu_15V_reg.kicad_pcb (KiCad board)
At the start: 2 copper layers, 55 x 50 mm, 24 parts, among them J1 IN, J2 OUT, U1 LM317_TO-252, U2 LM337_TO252

Commit message: rev2
Parts:
- moved D1 19.1 mm to (148.0, 94.5), turned to 270 degrees
- moved C2 16.1 mm to (127.0, 106.0)
- moved D2 13.5 mm to (124.8, 115.0), turned to 90 degrees
- moved C5 11.8 mm to (140.0, 84.8), turned to 90 degrees
- moved D3 9.51 mm to (144.0, 94.5), turned to 90 degrees
- moved C3 9.01 mm to (131.8, 84.5), turned to 180 degrees
- moved R3 8.71 mm to (133.0, 113.8), turned to 90 degrees
- moved C4 7.22 mm to (145.0, 107.2), turned to 0 degrees
- moved U2 6.86 mm to (143.8, 112.5)
- moved R4 6.09 mm to (136.0, 113.8)
- moved H1 5.71 mm to (106.2, 118.8)
- moved H2 5.26 mm to (156.2, 118.8)
- moved R1 4.83 mm to (136.8, 93.2), turned to 90 degrees
- moved U1 4.45 mm to (129.0, 90.2)
- moved R2 4.30 mm to (139.8, 93.2), turned to 270 degrees
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Routing:
- net /VO+: track 0.00 -> 28.9 mm
- net /VI-: track 0.00 -> 27.1 mm
- net /VO-: track 36.4 -> 45.2 mm
- net /VI+: track 33.4 -> 34.1 mm
- net GND: track 20.7 -> 20.4 mm, vias 69 -> 10
- removed copper zone on F.Cu, net /VO+
- removed copper zone on F.Cu, net GND
Other:
- board size 55 x 50 mm -> 57.5 x 45 mm
